File: headstage-neuropix_large-zif/headstage-neuropix.sch (EAGLE design)
At the start: 147 parts, among them J1 302-S101, J2 X.FL-R-SMT-1(02), J3 FH23-45S-0.3SHW(05), J5 77311-118-02LF, J6 FH23-45S-0.3SHW(05), U1 10M08SAM15317G, U10 PL133-27GC-R, U11 TS4231, U12 TS4231, U13 TS4231, U2 ASCO2-24.000MHZ-EK-T3, U3 MAX4945AELA+T, U4 DS90UB933_WQFN, U5 NCP161BMX330, U6 TPS8268180, U7 TLV70712, U8 BNO055, U9 DSC6102MI2A-093.6000, X2 OE-LOGO_14X10

Commit message: Updated BOM for revision 1.3
- External on google-sheet. Link added to READMEs for each board
version.
- Schematics updated to reflect the BOM.
- Added SMD mount information
- Added .gitignore and .gitattributes for LFS
Parts:
- removed C66: 10uF, jonnew:C_0402TW
- removed C67: 1uF, jonnew:C_0201T
- removed J6: FH23-45S-0.3SHW(05), jonnew:PINHD-1X45_FH23
- added C56: 10nF, jonnew:C_0201T
- added C60: 1uF, jonnew:C_0201T
- added J4: 77311-118-02LF, jonnew:JP2E_THRU-HOLE
- C24, C26, C28: value 0.1uF -> 10uF; device jonnew:C_0201T -> jonnew:C_0402TW
- C25: value 10uF -> 1uF; device jonnew:C_0402TW -> jonnew:C_0201T
- C27, C32: value 10uF -> 0.1uF; device jonnew:C_0402TW -> jonnew:C_0201T
- C30: value 10nF -> 1nF
- C31, C49: value 10nF -> 0.1uF
- C34, C40: value 0.1uF -> 10nF
- C36, C37: value 10nF -> 10uF; device jonnew:C_0201T -> jonnew:C_0402TW
- C38: value 0.1uF -> 1uF
- C41, C42: value 10uF -> 10nF; device jonnew:C_0402TW -> jonnew:C_0201T
- C43: value 0.1uF -> 1nF
- C44: value 47nF -> 0.1uF
- C45: value 4.7uF -> 0.1uF; device jonnew:C_0402T -> jonnew:C_0201T
- C46: value 10uF -> 0.1uF; device jonnew:C_0402T -> jonnew:C_0201T
- C48: value 1uF -> 10uF; device jonnew:C_0201T -> jonnew:C_0402TW
- C50: value 0.1uF -> 47nF
- C51: device jonnew:C_0402T -> jonnew:C_0402TW
- C52: value 10nF -> 4.7uF; device jonnew:C_0201T -> jonnew:C_0402T
- C53: value 1uF -> 10uF; device jonnew:C_0201T -> jonnew:C_0402T; PARTNO CL03A105MP3ZSNH -> (none)
- C54: value 1uF -> 10uF; device jonnew:C_0201T -> jonnew:C_0402TW; PARTNO CL03A105MP3ZSNH -> (none)
- C55: PARTNO CL03A105MP3ZSNH -> (none)
- C57: PARTNO C0603X5R1C104K030BC -> (none)
- C58: value 0.1uF -> 10uF; device jonnew:C_0201T -> jonnew:C_0402T; PARTNO C0603X5R1C104K030BC -> (none)
- C59: value 0.1uF -> 10nF; PARTNO C0603X5R1C104K030BC -> (none)
- C61: PARTNO (none) -> CL03A105MP3ZSNH
- C62: value 1nF -> 1uF; PARTNO (none) -> CL03A105MP3ZSNH
- C63: value 1nF -> 0.1uF; PARTNO (none) -> C0603X5R1C104K030BC
- C64, C65: value 10uF -> 0.1uF; device jonnew:C_0402TW -> jonnew:C_0201T; PARTNO (none) -> C0603X5R1C104K030BC
- J5: value 77311-118-02LF -> FH23-45S-0.3SHW(05); device jonnew:JP2E_THRU-HOLE -> jonnew:PINHD-1X45_FH23
- R21: value 49.9 -> 6.6k
- R23: value 10k -> 49.9
- R24: value 100k -> 10k
- R25: value 2k -> 10k
- R26: value 22 -> 100k
- R27: value 22 -> 2k
- R28: value 20k -> 22
- R29: value 100 -> 20k
- R30: value 15k -> 100
- R31: value 15k -> 22
- R33: value 20k -> 15k
- R34: value 100 -> 15k
- R35: value 6.6k -> 20k
- R36: value 10k -> 100
- U10: value PL133-27GC-R -> BNO055; device jonnew:CLKBUF2_DFN_2X1.3_PAD -> jonnew:BNO055
- U11: value TS4231 -> DSC6102MI2A-093.6000; device jonnew:TS4231 -> jonnew:CRYSTAL-OSC_VFLGA4-2X1.6
- U12: value TS4231 -> PL133-27GC-R; device jonnew:TS4231 -> jonnew:CLKBUF2_DFN_2X1.3_PAD
- U14, U15: value (none) -> TS4231; device jonnew:LDO_ADJUST-EN-SS_WLCSP-ADP7112 -> jonnew:TS4231
- U4: value DS90UB933_WQFN -> ADP7112ACBZ-1.8-R7; device jonnew:DS90UB913A_WQFN -> jonnew:LDO_ADJUST-EN-SS_WLCSP-ADP7112
- U5: value NCP161BMX330 -> DS90UB933_WQFN; device jonnew:TLV707 -> jonnew:DS90UB913A_WQFN
- U6: value TPS8268180 -> NCP161BMX330; device jonnew:TPS8268X -> jonnew:TLV707
- U7: value TLV70712 -> TPS8268180; device jonnew:TLV707 -> jonnew:TPS8268X
- U8: value BNO055 -> TLV70712; device jonnew:BNO055 -> jonnew:TLV707
- U9: value DSC6102MI2A-093.6000 -> ADP7112ACBZ-1.2-R7; device jonnew:CRYSTAL-OSC_VFLGA4-2X1.6 -> jonnew:LDO_ADJUST-EN-SS_WLCSP-ADP7112
- renumbered TP10 to TP8, TP13 to TP9
Connections:
- removed net N$9 (its old number): R30.2, U11.RBIAS
- new net N$29: R34.2, U15.RBIAS
- net !IMU_BL: now also R24.2, U10.!BOOT_LOAD; no longer R22.2, U8.!BOOT_LOAD
- net !IMU_RESET: now also R20.1, U10.!RESET; no longer R19.1, U8.!RESET
- net +1V2: now also C48.1, J5.P$38, J5.P$39, U8.OUT; no longer C42.1, J6.P$38, J6.P$39, U7.OUT
- net +1V8: now also C31.1, C34.1, C41.1, C45.1, C53.1, C56.2, C59.2, J5.P$42, J5.P$43, R25.1, U11.VCC, U12.EN, U12.VCC, U5.VDDD, U5.VDDT, U7.VOUT; no longer C28.1, C30.1, C36.1, C39.1, C46.1, C49.2, C52.2, J6.P$42, J6.P$43, R23.1, U10.EN, U10.VCC, U4.VDDD, U4.VDDT, U6.VOUT, U9.VCC
- net +3V3: now also C27.1, C32.1, C35.1, C37.1, C47.1, C63.1, C64.1, R20.2, R24.1, U10.VDD, U10.VDDIO, U14.DVDD, U15.DVDD, U4.VI, U5.VDDIO, U6.OUT, U8.EN, U8.IN, U9.VI; no longer C26.1, C31.1, C33.1, C41.1, C57.1, C58.1, C59.1, R19.2, R20.1, U11.DVDD, U12.DVDD, U14.VI, U15.VI, U4.VDDIO, U5.OUT, U7.EN, U7.IN, U8.VDD, U8.VDDIO
- net 1V2A: now also C51.1, J5.P$7, J5.P$8, U9.ADJ, U9.VO; no longer C66.1, J6.P$7, J6.P$8, U15.ADJ, U15.VO
- net 1V8A: now also C33.1, J5.P$3, J5.P$4, U4.ADJ, U4.VO; no longer C64.1, J6.P$3, J6.P$4, U14.ADJ, U14.VO
- net BNO_SCL: now also U10.COM1/SCL/RX; no longer U8.COM1/SCL/RX
- net BNO_SDA: now also U10.COM0/SDA/TX; no longer U8.COM0/SDA/TX
- net CAL_A_1KHZ: now also R29.1; no longer R28.1
- net CAL_B_1KHZ: now also R35.1; no longer R33.1
- net CAL_SIGNAL_A: now also R29.2, R30.1; no longer R28.2, R29.1
- net CAL_SIGNAL_A1: now also J5.P$11, R35.2, R36.1; no longer J6.P$11, R33.2, R34.1
- net GND: now also C34.2, C39.1, C43.2, C44.2, C52.2, C56.1, C59.1, C60.2, J4.2, J5.P$1, J5.P$10, J5.P$13, J5.P$14, J5.P$17, J5.P$2, J5.P$20, J5.P$23, J5.P$26, J5.P$29, J5.P$32, J5.P$34, J5.P$36, J5.P$37, J5.P$41, J5.P$44, J5.P$45, J5.P$5, J5.P$6, J5.P$9, R19.2, R23.1, R26.2, R30.2, R33.1, R34.1, U10.COM2, U10.COM3/ADDR, U10.GNDIO, U10.PS0, U10.PS1, U11.GND, U12.GND, U14.AVSS, U14.AVSS2, U15.AVSS, U15.AVSS2, U5.ID, U5.RES; no longer C34.1, C39.2, C49.1, C50.2, C52.1, C59.2, C66.2, C67.2, J5.2, J6.P$1, J6.P$10, J6.P$13, J6.P$14, J6.P$17, J6.P$2, J6.P$20, J6.P$23, J6.P$26, J6.P$29, J6.P$32, J6.P$34, J6.P$36, J6.P$37, J6.P$41, J6.P$44, J6.P$45, J6.P$5, J6.P$6, J6.P$9, R21.1, R24.2, R29.2, R30.1, R31.1, R34.2, U11.AVSS, U11.AVSS2, U12.AVSS, U12.AVSS2, U14.GND, U15.GND, U4.ID, U4.RES, U8.COM2, U8.COM3/ADDR, U8.GNDIO, U8.PS0, U8.PS1
- net I2C_SCL_B: now also J5.P$19; no longer J6.P$19
- net I2C_SDA_B: now also J5.P$18; no longer J6.P$18
- net LH_DATA0: now also U14.D/CFGDATA; no longer U12.D/CFGDATA
- net LH_DATA1: now also U13.D/CFGDATA; no longer U11.D/CFGDATA
- net LH_DATA2: now also U15.D/CFGDATA; no longer U13.D/CFGDATA
- net LH_ENV0: now also U14.E/CFGCLK; no longer U12.E/CFGCLK
- net LH_ENV1: now also U13.E/CFGCLK; no longer U11.E/CFGCLK
- net LH_ENV2: now also U15.E/CFGCLK; no longer U13.E/CFGCLK
- net MIDFILT: now also R27.1; no longer R25.1
- net N$1: now also U11.OUT, U12.IN; no longer U10.IN, U9.OUT
- net N$12: now also C60.1, U13.AVDD; no longer C53.1, U11.AVDD
- net N$13: now also C58.1, R27.2; no longer C51.1, R25.2
- net N$14: now also U14.IIN-; no longer U12.IIN-
- net N$15: now also U14.IIN+; no longer U12.IIN+
- net N$16: now also R33.2, U14.RBIAS; no longer R31.2, U12.RBIAS
- net N$2: now also R28.1, U12.CLK0; no longer R26.1, U10.CLK0
- net N$26: now also U15.IIN-; no longer U13.IIN-
- net N$27: now also U15.IIN+; no longer U13.IIN+
- net N$28: now also C49.2, U5.DOUT+; no longer C43.2, U4.DOUT+
- net N$3: now also R31.2; no longer R27.2
- net N$30: now also C55.1, R22.2, U5.PDB; no longer C48.1, R20.2, U4.PDB
- net N$31: now also C50.2, U5.DOUT-; no longer C44.2, U4.DOUT-
- net N$32: now also C50.1, R23.2; no longer C44.1, R21.2
- net N$33: now also C57.1, R25.2, R26.1, U5.MODE; no longer C50.1, R23.2, R24.1, U4.MODE
- net N$34: now also C40.1, C44.1, C52.1, U5.VDDPLL; no longer C35.1, C38.1, C45.1, U4.VDDPLL
- net N$35: now also C42.1, C46.1, C54.1, U5.VDDCML; no longer C37.1, C40.1, C47.1, U4.VDDCML
- net N$36: now also C61.1, U14.AVDD; no longer C54.1, U12.AVDD
- net N$37: now also C62.1, U15.AVDD; no longer C55.1, U13.AVDD
- net N$38: now also C26.1, C28.1, C36.1, U6.IN, U7.EN, U7.MODE, U7.VIN; no longer C25.1, C27.1, C32.1, U5.EN, U5.IN, U6.MODE, U6.VIN
- net N$39: now also C30.1, U4.SS; no longer C62.1, U14.SS
- net N$40: now also C43.1, U9.SS; no longer C63.1, U15.SS
- net N$41: now also C38.1, R21.1, U9.EN; no longer C67.1, R35.1, U15.EN
- net N$5: now also J5.P$35, R28.2; no longer J6.P$35, R26.2
- net N$6: now also R31.1, U12.CLK1; no longer R27.1, U10.CLK1
- net N$67: now also C39.2, U10.CAP; no longer C34.2, U8.CAP
- net N$7: now also U13.IIN-; no longer U11.IIN-
- net N$8: now also U13.IIN+; no longer U11.IIN+
- net NP_OSC_EN: now also U11.EN; no longer U9.EN
- net NRST: now also J5.P$15, R21.2, U4.EN; no longer J6.P$15, R35.2, U14.EN
- net OSC_PDOWN_N_B: now also J5.P$12; no longer J6.P$12
- net PSB_CLK_B: now also J5.P$33; no longer J6.P$33
- net PSB_DATA_0_B: now also J5.P$31; no longer J6.P$31
- net PSB_DATA_1_B: now also J5.P$30; no longer J6.P$30
- net PSB_DATA_2_B: now also J5.P$28; no longer J6.P$28
- net PSB_DATA_3_B: now also J5.P$27; no longer J6.P$27
- net PSB_DATA_4_B: now also J5.P$25; no longer J6.P$25
- net PSB_DATA_5_B: now also J5.P$24; no longer J6.P$24
- net PSB_DATA_6_B: now also J5.P$22; no longer J6.P$22
- net PSB_SYNC_B: now also J5.P$21; no longer J6.P$21
- net REC_NRST_B: now also J5.P$16; no longer J6.P$16
- net SER_DIN0: now also U5.DIN0; no longer U4.DIN0
- net SER_DIN1: now also U5.DIN1; no longer U4.DIN1
- net SER_DIN10: now also U5.DIN10; no longer U4.DIN10
- net SER_DIN11: now also U5.DIN11; no longer U4.DIN11
- net SER_DIN2: now also U5.DIN2; no longer U4.DIN2
- net SER_DIN3: now also U5.DIN3; no longer U4.DIN3
- net SER_DIN4: now also U5.DIN4; no longer U4.DIN4
- net SER_DIN5: now also U5.DIN5; no longer U4.DIN5
- net SER_DIN6: now also U5.DIN6; no longer U4.DIN6
- net SER_DIN7: now also U5.DIN7; no longer U4.DIN7
- net SER_DIN8: now also U5.DIN8; no longer U4.DIN8
- net SER_DIN9: now also U5.DIN9; no longer U4.DIN9
- net SER_GPIO0: now also U5.GPIO0; no longer U4.GPIO0
- net SER_GPIO1: now also U5.GPIO1; no longer U4.GPIO1
- net SER_GPIO2: now also R19.1, U5.GPIO2/CLKOUT; no longer R36.1, U4.GPIO2/CLKOUT
- net SER_GPIO3: now also U5.GPO3/CLKIN; no longer U4.GPO3/CLKIN
- net SER_HSYNC: now also U5.HSYNC; no longer U4.HSYNC
- net SER_PCLK: now also U5.PCLK1; no longer U4.PCLK1
- net SER_SCL: now also U5.SCL; no longer U4.SCL
- net SER_SDA: now also U5.SDA; no longer U4.SDA
- net SER_VSYNC: now also U5.VSYNC; no longer U4.VSYNC
- net SIGOUT: now also C49.1; no longer C43.1
- net VCOAX: now also C25.1, J4.1; no longer C61.1, J5.1
Other:
- moved on the sheet: C24, C25, C26, C27, C28, C29, C30, C31, C32, C33, C34, C35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
