File: headstage-neuropix_standard-zif/headstage-neuropix.sch (EAGLE design)
At the start: 147 parts, among them J1 302-S101, J2 X.FL-R-SMT-1(02), J3 1-2013496-8, J4 77311-118-02LF, J5 1-2013496-8, U1 10M08SAM15317G, U10 BNO055, U11 DSC6102MI2A-093.6000, U12 PL133-27GC-R, U13 TS4231, U14 TS4231, U15 TS4231, U2 ASCO2-24.000MHZ-EK-T3, U3 MAX4945AELA+T, U4 ADP7112ACBZ-1.8-R7, U5 DS90UB933_WQFN, U6 NCP161BMX330, U7 TPS8268180, U8 TLV70712, U9 ADP7112ACBZ-1.2-R7, X2 OE-LOGO_14X10

Commit message: Correct tPlace/tStop mixup for ADP7112's
- Solder pads had tPlace instead of tStop so there would have been
silkscreen on the pads
Parts:
- U10: value BNO055 -> BNO055_LP; device jonnew:BNO055 -> jonnew:BNO055_LP
- U4, U9: device jonnew:LDO_ADJUST-EN-SS_WLCSP-ADP7112 -> jonnew:LDO_ADJUST-EN-SS_WLCSP-ADP7112_LP
- U5: device jonnew:DS90UB913A_WQFN -> jonnew:DS90UB913A_LP
Changed lines of the file:
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@@
 </classes>
 <parts>
-<part name="U5" library="jonnew" deviceset="DS90UB913A" device="_WQFN" value="DS90UB933_WQFN"/>
+<part name="U5" library="jonnew" deviceset="DS90UB913A" device="_LP" value="DS90UB933_WQFN"/>
 <part name="U6" library="jonnew" deviceset="TLV707" device="" value="NCP161BMX330"/>
 <part name="U8" library="jonnew" deviceset="TLV707" device="" value="TLV70712"/>
@@
 <part name="SUPPLY29" library="jonnew" deviceset="GND" device=""/>
 <part name="P29" library="jonnew" deviceset="+3V3" device=""/>
-<part name="U10" library="jonnew" deviceset="BNO055" device=""/>
+<part name="U10" library="jonnew" deviceset="BNO055" device="_LP" value="BNO055_LP"/>
 <part name="C39" library="jonnew" deviceset="C" device="_0201T" value="0.1uF"/>
 <part name="SUPPLY20" library="jonnew" deviceset="GND" device=""/>
@@
 <part name="SUPPLY21" library="jonnew" deviceset="GND" device=""/>
 <part name="C25" library="jonnew" deviceset="C" device="_0201T" value="1uF"/>
-<part name="U4" library="jonnew" deviceset="LDO_ADJUST-EN-SS" device="_WLCSP-ADP7112" value="ADP7112ACBZ-1.8-R7"/>
-<part name="U9" library="jonnew" deviceset="LDO_ADJUST-EN-SS" device="_WLCSP-ADP7112" value="ADP7112ACBZ-1.2-R7"/>
+<part name="U4" library="jonnew" deviceset="LDO_ADJUST-EN-SS" device="_WLCSP-ADP7112_LP" value="ADP7112ACBZ-1.8-R7"/>
+<part name="U9" library="jonnew" deviceset="LDO_ADJUST-EN-SS" device="_WLCSP-ADP7112_LP" value="ADP7112ACBZ-1.2-R7"/>
 <part name="C30" library="jonnew" deviceset="C" device="_0201T" value="1nF"/>
 <part name="C33" library="jonnew" deviceset="C" device="_0402TW" value="10uF"/>
@@
 the external 32.768 kHz crystal.</text>
 <wire x1="248.92" y1="264.16" x2="248.92" y2="469.9" width="0.508" layer="94" style="longdash"/>
-<wire x1="248.92" y1="469.9" x2="248.92" y2="612.14" width="0.508" layer="94" style="longdash"/>
-<wire x1="248.92" y1="612.14" x2="248.92" y2="835.66" width="0.508" layer="94" style="longdash"/>
+<wire x1="248.92" y1="469.9" x2="248.92" y2="601.98" width="0.508" layer="94" style="longdash"/>
+<wire x1="248.92" y1="601.98" x2="248.92" y2="835.66" width="0.508" layer="94" style="longdash"/>
 <wire x1="248.92" y1="469.9" x2="477.52" y2="469.9" width="0.508" layer="94" style="longdash"/>
-<wire x1="248.92" y1="612.14" x2="421.64" y2="612.14" width="0.508" layer="94" style="longdash"/>
-<wire x1="421.64" y1="612.14" x2="477.52" y2="612.14" width="0.508" layer="94" style="longdash"/>
-<wire x1="477.52" y1="612.14" x2="721.36" y2="612.14" width="0.508" layer="94" style="longdash"/>
-<wire x1="477.52" y1="612.14" x2="477.52" y2="469.9" width="0.508" layer="94" style="longdash"/>
+<wire x1="248.92" y1="601.98" x2="421.64" y2="601.98" width="0.508" layer="94" style="longdash"/>
+<wire x1="421.64" y1="601.98" x2="477.52" y2="601.98" width="0.508" layer="94" style="longdash"/>
+<wire x1="477.52" y1="601.98" x2="721.36" y2="601.98" width="0.508" layer="94" style="longdash"/>
+<wire x1="477.52" y1="601.98" x2="477.52" y2="469.9" width="0.508" layer="94" style="longdash"/>
 <wire x1="477.52" y1="469.9" x2="477.52" y2="393.7" width="0.508" layer="94" style="longdash"/>
-<wire x1="421.64" y1="612.14" x2="421.64" y2="835.66" width="0.508" layer="94" style="longdash"/>
+<wire x1="421.64" y1="601.98" x2="421.64" y2="835.66" width="0.508" layer="94" style="longdash"/>
 <text x="525.78" y="457.2" size="10.16" layer="97" rot="R90">3D TRACKING</text>
 <wire x1="477.52" y1="393.7" x2="591.82" y2="393.7" width="0.508" layer="94" style="longdash"/>
